Commit message: [FEAT] Change realsense xacro harcoded values to parameters

File: xarm_description/urdf/camera/realsense_d435i.urdf.xacro (robot description, xacro)
@@ -1,13 +1,13 @@
 <?xml version="1.0"?>
 <robot xmlns:xacro="http://ros.org/wiki/xacro">
-  <xacro:macro name="d435i_urdf" params="prefix:='' add_d435i_links:=false">
+  <xacro:macro name="d435i_urdf" params="prefix:='' identifier:='' parent_link:='link_eef' add_d435i_links:=false  xyz:='0.06746 -0.0175 0.0237' rpy:='3.1415926535897931 ${-3.1415926535897931/2} 0'">
     <!-- define property -->
     <xacro:property name="M_PI" value="3.1415926535897931" />
-    <link name="${prefix}link_eef">
+    <link name="${prefix}${parent_link}">
       <xacro:common_link_visual
         mesh_filename="camera/realsense/visual/d435_with_cam_stand"
         origin_xyz="0 0 0"
         origin_rpy="0 0 0"
-        material_name="${prefix}Silver" />
+        material_name="Silver" />
       <xacro:common_link_collision
         mesh_filename="camera/realsense/collision/d435_with_cam_stand"
@@ -16,56 +16,56 @@
     </link>
     <xacro:if value="${add_d435i_links}">
-      <link name="${prefix}camera_link"></link>
-      <link name="${prefix}camera_depth_frame"></link>
-      <link name="${prefix}camera_depth_optical_frame"></link>
-      <link name="${prefix}camera_color_frame"></link>
-      <link name="${prefix}camera_color_optical_frame"></link>
-      <link name="${prefix}camera_left_ir_frame"></link>
-      <link name="${prefix}camera_left_ir_optical_frame"></link>
-      <link name="${prefix}camera_right_ir_frame"></link>
-      <link name="${prefix}camera_right_ir_optical_frame"></link>
-      <joint name="${prefix}camera_link_joint" type="fixed">
-        <parent link="${prefix}link_eef" />
-        <child link="${prefix}camera_link" />
-        <origin xyz="0.06746 -0.0175 0.0237" rpy="${M_PI} ${-M_PI/2} 0" />
+      <link name="${prefix}${identifier}camera_link"></link>
+      <link name="${prefix}${identifier}camera_depth_frame"></link>
+      <link name="${prefix}${identifier}camera_depth_optical_frame"></link>
+      <link name="${prefix}${identifier}camera_color_frame"></link>
+      <link name="${prefix}${identifier}camera_color_optical_frame"></link>
+      <link name="${prefix}${identifier}camera_left_ir_frame"></link>
+      <link name="${prefix}${identifier}camera_left_ir_optical_frame"></link>
+      <link name="${prefix}${identifier}camera_right_ir_frame"></link>
+      <link name="${prefix}${identifier}camera_right_ir_optical_frame"></link>
+      <joint name="${prefix}${identifier}camera_link_joint" type="fixed">
+        <parent link="${prefix}${identifier}${parent_link}" />
+        <child link="${prefix}${identifier}camera_link" />
+        <origin xyz="${xyz}" rpy="${rpy}" />
       </joint>
-      <joint name="${prefix}camera_depth_joint" type="fixed">
-        <parent link="${prefix}camera_link" />
-        <child link="${prefix}camera_depth_frame" />
+      <joint name="${prefix}${identifier}camera_depth_joint" type="fixed">
+        <parent link="${prefix}${identifier}camera_link" />
+        <child link="${prefix}${identifier}camera_depth_frame" />
         <origin xyz="0 0 0" rpy="0 0 0" />
       </joint>
-      <joint name="${prefix}camera_depth_optical_joint" type="fixed">
-        <parent link="${prefix}camera_depth_frame" />
-        <child link="${prefix}camera_depth_optical_frame" />
+      <joint name="${prefix}${identifier}camera_depth_optical_joint" type="fixed">
+        <parent link="${prefix}${identifier}camera_depth_frame" />
+        <child link="${prefix}${identifier}camera_depth_optical_frame" />
         <origin xyz="0 0 0" rpy="${-M_PI/2} 0 ${-M_PI/2}" />
       </joint>
-      <joint name="${prefix}camera_color_joint" type="fixed">
-        <parent link="${prefix}camera_link" />
-        <child link="${prefix}camera_color_frame" />
+      <joint name="${prefix}${identifier}camera_color_joint" type="fixed">
+        <parent link="${prefix}${identifier}camera_link" />
+        <child link="${prefix}${identifier}camera_color_frame" />
         <origin xyz="0 0.015 0" rpy="0 0 0" />
       </joint>
-      <joint name="${prefix}camera_color_optical_joint" type="fixed">
-        <parent link="${prefix}camera_color_frame" />
-        <child link="${prefix}camera_color_optical_frame" />
+      <joint name="${prefix}${identifier}camera_color_optical_joint" type="fixed">
+        <parent link="${prefix}${identifier}camera_color_frame" />
+        <child link="${prefix}${identifier}camera_color_optical_frame" />
         <origin xyz="0 0 0" rpy="${-M_PI/2} 0 ${-M_PI/2}" />
       </joint>
-      <joint name="${prefix}camera_left_ir_joint" type="fixed">
-        <parent link="${prefix}camera_link" />
-        <child link="${prefix}camera_left_ir_frame" />
+      <joint name="${prefix}${identifier}camera_left_ir_joint" type="fixed">
+        <parent link="${prefix}${identifier}camera_link" />
+        <child link="${prefix}${identifier}camera_left_ir_frame" />
         <origin xyz="0 0 0" rpy="0 0 0" />
       </joint>
-      <joint name="${prefix}camera_left_ir_optical_joint" type="fixed">
-        <parent link="${prefix}camera_left_ir_frame" />
-        <child link="${prefix}camera_left_ir_optical_frame" />
+      <joint name="${prefix}${identifier}camera_left_ir_optical_joint" type="fixed">
+        <parent link="${prefix}${identifier}camera_left_ir_frame" />
+        <child link="${prefix}${identifier}camera_left_ir_optical_frame" />
         <origin xyz="0 0 0" rpy="${-M_PI/2} 0 ${-M_PI/2}" />
       </joint>
-      <joint name="${prefix}camera_right_ir_joint" type="fixed">
-        <parent link="${prefix}camera_link" />
-        <child link="${prefix}camera_right_ir_frame" />
+      <joint name="${prefix}${identifier}camera_right_ir_joint" type="fixed">
+        <parent link="${prefix}${identifier}camera_link" />
+        <child link="${prefix}${identifier}camera_right_ir_frame" />
         <origin xyz="0 -0.050 0" rpy="0 0 0" />
       </joint>
-      <joint name="${prefix}camera_right_ir_optical_joint" type="fixed">
-        <parent link="${prefix}camera_right_ir_frame" />
-        <child link="${prefix}camera_right_ir_optical_frame" />
+      <joint name="${prefix}${identifier}camera_right_ir_optical_joint" type="fixed">
+        <parent link="${prefix}${identifier}camera_right_ir_frame" />
+        <child link="${prefix}${identifier}camera_right_ir_optical_frame" />
         <origin xyz="0 0 0" rpy="${-M_PI/2} 0 ${-M_PI/2}" />
       </joint>
