Commit message: [FEAT] Add parameters to support external cameras

File: xarm_description/urdf/camera/realsense.gazebo.xacro (robot description, xacro)
@@ -1,6 +1,13 @@
 <?xml version="1.0"?>
 <robot xmlns:xacro="http://ros.org/wiki/xacro">
-  <xacro:macro name="realsense_gazebo" params="prefix:='' ">
-    <gazebo reference="${prefix}camera_depth_frame">
+  <xacro:macro name="realsense_gazebo" params="prefix:='' identifier:=''">
+   <!-- define property -->
+    <xacro:if value="${identifier == ''}">
+      <xacro:property name="camera_name" value="${prefix}" />
+    </xacro:if>
+    <xacro:if value="${identifier != ''}">
+      <xacro:property name="camera_name" value="${prefix}${identifier}_" />
+    </xacro:if>
+    <gazebo reference="${camera_name}camera_depth_frame">
       <sensor name="cameradepth" type="depth">
         <camera name="camera">
@@ -25,5 +32,5 @@
       </sensor>
     </gazebo>
-    <gazebo reference="${prefix}camera_color_frame">
+    <gazebo reference="${camera_name}camera_color_frame">
       <sensor name="cameracolor" type="camera">
         <camera name="camera">
@@ -49,5 +56,5 @@
       </sensor>
     </gazebo>
-    <gazebo reference="${prefix}camera_left_ir_frame">
+    <gazebo reference="${camera_name}camera_left_ir_frame">
       <sensor name="cameraired1" type="camera">
         <camera name="camera">
@@ -73,5 +80,5 @@
       </sensor>
     </gazebo>
-    <gazebo reference="${prefix}camera_right_ir_frame">
+    <gazebo reference="${camera_name}camera_right_ir_frame">
       <sensor name="cameraired2" type="camera">
         <camera name="camera">

File: xarm_description/urdf/camera/realsense_d435i.urdf.xacro (robot description, xacro)
@@ -1,7 +1,12 @@
 <?xml version="1.0"?>
 <robot xmlns:xacro="http://ros.org/wiki/xacro">
-  <xacro:macro name="d435i_urdf" params="prefix:='' identifier:='' parent_link:='link_eef' add_d435i_links:=false  xyz:='0.06746 -0.0175 0.0237' rpy:='3.1415926535897931 ${-3.1415926535897931/2} 0'">
+  <xacro:macro name="d435i_urdf" params="prefix:='' identifier:='' parent_link:='link_eef' add_d435i_links:=false">
     <!-- define property -->
-    <xacro:property name="M_PI" value="3.1415926535897931" />
+    <xacro:if value="${identifier == ''}">
+    <xacro:property name="camera_name" value="${prefix}" />
+    </xacro:if>
+    <xacro:if value="${identifier != ''}">
+    <xacro:property name="camera_name" value="${prefix}${identifier}_" />
+    </xacro:if>
     <link name="${prefix}${parent_link}">
       <xacro:common_link_visual
@@ -16,57 +21,57 @@
     </link>
     <xacro:if value="${add_d435i_links}">
-      <link name="${prefix}${identifier}camera_link"></link>
-      <link name="${prefix}${identifier}camera_depth_frame"></link>
-      <link name="${prefix}${identifier}camera_depth_optical_frame"></link>
-      <link name="${prefix}${identifier}camera_color_frame"></link>
-      <link name="${prefix}${identifier}camera_color_optical_frame"></link>
-      <link name="${prefix}${identifier}camera_left_ir_frame"></link>
-      <link name="${prefix}${identifier}camera_left_ir_optical_frame"></link>
-      <link name="${prefix}${identifier}camera_right_ir_frame"></link>
-      <link name="${prefix}${identifier}camera_right_ir_optical_frame"></link>
-      <joint name="${prefix}${identifier}camera_link_joint" type="fixed">
-        <parent link="${prefix}${identifier}${parent_link}" />
-        <child link="${prefix}${identifier}camera_link" />
-        <origin xyz="${xyz}" rpy="${rpy}" />
+      <link name="${camera_name}camera_link"></link>
+      <link name="${camera_name}camera_depth_frame"></link>
+      <link name="${camera_name}camera_depth_optical_frame"></link>
+      <link name="${camera_name}camera_color_frame"></link>
+      <link name="${camera_name}camera_color_optical_frame"></link>
+      <link name="${camera_name}camera_left_ir_frame"></link>
+      <link name="${camera_name}camera_left_ir_optical_frame"></link>
+      <link name="${camera_name}camera_right_ir_frame"></link>
+      <link name="${camera_name}camera_right_ir_optical_frame"></link>
+      <joint name="${camera_name}camera_link_joint" type="fixed">
+        <parent link="${prefix}${parent_link}" />
+        <child link="${camera_name}camera_link" />
+        <origin xyz="0.06746 -0.0175 0.0237" rpy="${pi} ${-pi/2} 0" />
       </joint>
-      <joint name="${prefix}${identifier}camera_depth_joint" type="fixed">
-        <parent link="${prefix}${identifier}camera_link" />
-        <child link="${prefix}${identifier}camera_depth_frame" />
+      <joint name="${camera_name}camera_depth_joint" type="fixed">
+        <parent link="${camera_name}camera_link" />
+        <child link="${camera_name}camera_depth_frame" />
         <origin xyz="0 0 0" rpy="0 0 0" />
       </joint>
-      <joint name="${prefix}${identifier}camera_depth_optical_joint" type="fixed">
-        <parent link="${prefix}${identifier}camera_depth_frame" />
-        <child link="${prefix}${identifier}camera_depth_optical_frame" />
-        <origin xyz="0 0 0" rpy="${-M_PI/2} 0 ${-M_PI/2}" />
+      <joint name="${camera_name}camera_depth_optical_joint" type="fixed">
+        <parent link="${camera_name}camera_depth_frame" />
+        <child link="${camera_name}camera_depth_optical_frame" />
+        <origin xyz="0 0 0" rpy="${-pi/2} 0 ${-pi/2}" />
       </joint>
-      <joint name="${prefix}${identifier}camera_color_joint" type="fixed">
-        <parent link="${prefix}${identifier}camera_link" />
-        <child link="${prefix}${identifier}camera_color_frame" />
+      <joint name="${camera_name}camera_color_joint" type="fixed">
+        <parent link="${camera_name}camera_link" />
+        <child link="${camera_name}camera_color_frame" />
         <origin xyz="0 0.015 0" rpy="0 0 0" />
       </joint>
-      <joint name="${prefix}${identifier}camera_color_optical_joint" type="fixed">
-        <parent link="${prefix}${identifier}camera_color_frame" />
-        <child link="${prefix}${identifier}camera_color_optical_frame" />
-        <origin xyz="0 0 0" rpy="${-M_PI/2} 0 ${-M_PI/2}" />
+      <joint name="${camera_name}camera_color_optical_joint" type="fixed">
+        <parent link="${camera_name}camera_color_frame" />
+        <child link="${camera_name}camera_color_optical_frame" />
+        <origin xyz="0 0 0" rpy="${-pi/2} 0 ${-pi/2}" />
       </joint>
-      <joint name="${prefix}${identifier}camera_left_ir_joint" type="fixed">
-        <parent link="${prefix}${identifier}camera_link" />
-        <child link="${prefix}${identifier}camera_left_ir_frame" />
+      <joint name="${camera_name}camera_left_ir_joint" type="fixed">
+        <parent link="${camera_name}camera_link" />
+        <child link="${camera_name}camera_left_ir_frame" />
         <origin xyz="0 0 0" rpy="0 0 0" />
       </joint>
-      <joint name="${prefix}${identifier}camera_left_ir_optical_joint" type="fixed">
-        <parent link="${prefix}${identifier}camera_left_ir_frame" />
-        <child link="${prefix}${identifier}camera_left_ir_optical_frame" />
-        <origin xyz="0 0 0" rpy="${-M_PI/2} 0 ${-M_PI/2}" />
+      <joint name="${camera_name}camera_left_ir_optical_joint" type="fixed">
+        <parent link="${camera_name}camera_left_ir_frame" />
+        <child link="${camera_name}camera_left_ir_optical_frame" />
+        <origin xyz="0 0 0" rpy="${-pi/2} 0 ${-pi/2}" />
       </joint>
-      <joint name="${prefix}${identifier}camera_right_ir_joint" type="fixed">
-        <parent link="${prefix}${identifier}camera_link" />
-        <child link="${prefix}${identifier}camera_right_ir_frame" />
+      <joint name="${camera_name}camera_right_ir_joint" type="fixed">
+        <parent link="${camera_name}camera_link" />
+        <child link="${camera_name}camera_right_ir_frame" />
         <origin xyz="0 -0.050 0" rpy="0 0 0" />
       </joint>
-      <joint name="${prefix}${identifier}camera_right_ir_optical_joint" type="fixed">
-        <parent link="${prefix}${identifier}camera_right_ir_frame" />
-        <child link="${prefix}${identifier}camera_right_ir_optical_frame" />
-        <origin xyz="0 0 0" rpy="${-M_PI/2} 0 ${-M_PI/2}" />
+      <joint name="${camera_name}camera_right_ir_optical_joint" type="fixed">
+        <parent link="${camera_name}camera_right_ir_frame" />
+        <child link="${camera_name}camera_right_ir_optical_frame" />
+        <origin xyz="0 0 0" rpy="${-pi/2} 0 ${-pi/2}" />
       </joint>
     </xacro:if>
